Commit message: Wrote the framework for jacobian control
Former-commit-id: a5f1fb7982545c3c734fd81c56efbd5a91d5f2db

File: compliance/scenes/Krang.urdf (robot description, URDF)
Before this commit: robot Krang, 25 links, 24 joints
Links:
- link LFT: geometry collision box size=0.077 0.0962 0.077; visual mesh filename=Schunk/L7.dae
- link RFT: geometry collision box size=0.077 0.0962 0.077; visual mesh filename=Schunk/L7.dae
- link lGripper: geometry collision box size=0.1120 0.093 0.0800; visual mesh filename=Schunk/gripper.dae
- link rGripper: geometry collision box size=0.1120 0.093 0.0800; visual mesh filename=Schunk/gripper.dae
Joints:
- joint LMotorGripper: origin xyz=0.0 -0.035 0 rpy=3.1416 0 0 -> xyz=0 -0.0672 0 rpy=3.1416 0 0
- joint LMotorPlate1: origin xyz=-0.0 0.028 0.0 rpy=1.57 0.0 0 -> xyz=-0.0 0.1 0.0 rpy=1.57 0.0 0
- joint LMotorPlate2: origin xyz=0.025 0.028 0.0 rpy=1.57 3.1416 0 -> xyz=0.045 0.1 0.0 rpy=1.57 3.1416 0
- joint RMotorGripper: origin xyz=0 -0.035 0 rpy=3.1416 0 0 -> xyz=0 -0.0672 0 rpy=3.1416 0 0
- joint RMotorPlate1: origin xyz=-0.0 0.028 0.0 rpy=1.57 0.0 0 -> xyz=-0.0 0.100 0.0 rpy=1.57 0.0 0
- joint RMotorPlate2: origin xyz=0.025 0.028 0.0 rpy=1.57 3.1416 0 -> xyz=0.045 0.1 0.0 rpy=1.57 3.1416 0

File: compliance/scenes/KrangBlocks.urdf (robot description, URDF)
Before this commit: robot Krang, 25 links, 24 joints
Links:
- link LFT: geometry collision box size=0.077 0.0962 0.077; visual box size=0.077 0.0962 0.077
- link RFT: geometry collision box size=0.077 0.0962 0.077; visual box size=0.077 0.0962 0.077
- link lGripper: geometry collision box size=0.1120 0.093 0.0800; visual box size=0.1120 0.093 0.0800
- link rGripper: geometry collision box size=0.1120 0.093 0.0800; visual box size=0.1120 0.093 0.0800
Joints:
- joint LMotorGripper: origin xyz=0.0 -0.035 0 rpy=3.1416 0 0 -> xyz=0.0 -0.0672 0 rpy=3.1416 0 0
- joint LMotorPlate1: origin xyz=-0.025 0.028 0.0 rpy=1.57 0.0 0 -> xyz=-0.050 0.1 0.0 rpy=1.57 0.0 0
- joint LMotorPlate2: origin xyz=0.025 0.028 0.0 rpy=1.57 3.1416 0 -> xyz=0.050 0.1 0.0 rpy=1.57 3.1416 0
- joint RMotorGripper: origin xyz=0 -0.035 0 rpy=3.1416 0 0 -> xyz=0 -0.0672 0 rpy=3.1416 0 0
- joint RMotorPlate1: origin xyz=-0.025 0.028 0.0 rpy=1.57 0.0 0 -> xyz=-0.050 0.1 0.0 rpy=1.57 0.0 0
- joint RMotorPlate2: origin xyz=0.025 0.028 0.0 rpy=1.57 3.1416 0 -> xyz=0.050 0.1 0.0 rpy=1.57 3.1416 0

Commit message: Changed the dart model to incorporate the twist in the gripper and tested dart kinematics on correction. Next: estimation, then: fix frame in compliance
Former-commit-id: dd8b10d6a96664ea990cc81439ba883f65c05c6d

File: compliance/scenes/Krang.urdf (robot description, URDF)
Before this commit: robot Krang, 25 links, 24 joints
Links:
- removed link LFT
- removed link RFT
- link lGripper: mass None -> 1.206; geometry collision box size=0.08 0.112 0.2025; visual mesh filename=Schunk/L7.dae
- link rGripper: mass None -> 1.206; geometry collision box size=0.08 0.112 0.2025; visual mesh filename=Schunk/L7.dae
Joints:
- removed joint LMotorGripper
- removed joint RMotorGripper
- joint LJFT: child LFT -> lGripper; origin xyz=0 -0.159 0 rpy=0 0 0 -> xyz=0 -0.200 0 rpy=1.5708 3.1416 0
- joint LMotorPlate1: limit lower=0.0 upper=0.0135 effort=1000 velocity=0.1 -> lower=0.0 upper=0.022 effort=1000 velocity=0.1; origin xyz=-0.0 0.1 0.0 rpy=1.57 0.0 0 -> xyz=0.02043 -0.04010 0.127 rpy=3.1416 0 2.04; type fixed -> prismatic
- joint LMotorPlate2: limit lower=0.0 upper=0.0135 effort=1000 velocity=0.1 -> lower=0.0 upper=0.022 effort=1000 velocity=0.1; origin xyz=0.045 0.1 0.0 rpy=1.57 3.1416 0 -> xyz=-0.02043 0.04010 0.127 rpy=3.1416 0 -1.10; type fixed -> prismatic
- joint RJFT: child RFT -> rGripper; origin xyz=0 -0.159 0 rpy=0 0 0 -> xyz=0 -0.200 0 rpy=1.5708 3.1416 0
- joint RMotorPlate1: limit lower=0.0 upper=0.0135 effort=1000 velocity=0.1 -> lower=0.0 upper=0.022 effort=1000 velocity=0.1; origin xyz=-0.0 0.100 0.0 rpy=1.57 0.0 0 -> xyz=0.02043 -0.04010 0.127 rpy=3.1416 0 2.04
- joint RMotorPlate2: limit lower=0.0 upper=0.0135 effort=1000 velocity=0.1 -> lower=0.0 upper=0.022 effort=1000 velocity=0.1; origin xyz=0.045 0.1 0.0 rpy=1.57 3.1416 0 -> xyz=-0.02043 0.04010 0.127 rpy=3.1416 0 -1.10

File: compliance/scenes/KrangBlocks.urdf (robot description, URDF)
Before this commit: robot Krang, 25 links, 24 joints
Links:
- removed link LFT
- removed link RFT
- link lGripper: mass None -> 1.206; geometry collision box size=0.08 0.112 0.2025; visual box size=0.08 0.112 0.2025
- link rGripper: mass None -> 1.206; geometry collision box size=0.08 0.112 0.2025; visual box size=0.08 0.112 0.2025
Joints:
- removed joint LMotorGripper
- removed joint RMotorGripper
- joint LJFT: child LFT -> lGripper; origin xyz=0 -0.159 0 rpy=0 0 0 -> xyz=0 -0.200 0 rpy=1.5708 3.1416 0
- joint LMotorPlate1: origin xyz=-0.050 0.1 0.0 rpy=1.57 0.0 0 -> xyz=0.02043 -0.04010 0.127 rpy=3.1416 0 2.04
- joint LMotorPlate2: origin xyz=0.050 0.1 0.0 rpy=1.57 3.1416 0 -> xyz=-0.02043 0.04010 0.127 rpy=3.1416 0 -1.10
- joint RJFT: child RFT -> rGripper; limit lower=-6.2832 upper=6.2832 effort=1000 velocity=0.1 -> lower=-3.1416 upper=3.1416 effort=1000 velocity=0.1; origin xyz=0 -0.159 0 rpy=0 0 0 -> xyz=0 -0.200 0 rpy=1.5708 3.1416 0
- joint RMotorPlate1: origin xyz=-0.050 0.1 0.0 rpy=1.57 0.0 0 -> xyz=-0.02043 0.04010 0.127 rpy=3.1416 0 -1.10

File: compliance/scenes/testObject.urdf (robot description, URDF)
Before this commit: robot cylinder, 1 links, 0 joints
Links:
- link base_link: geometry collision box size=0.08 0.112 0.2025; visual mesh filename=Schunk/L7.dae
