Commit message: Got some compliance going. two problems: (1) frame error and (2) jerkiness (maybe due frame?)
Former-commit-id: 16333f32c4cd8bf9b47289a0779d0eccbea1f91d

File: compliance/scenes/KrangBlocks.urdf (robot description, URDF)
Before this commit: robot Krang, 25 links, 24 joints
Joints:
- joint LMotorGripper: origin xyz=0.0 -0.0672 0 rpy=3.1416 0 0 -> xyz=0.0 -0.0672 0 rpy=3.1416 0.7854 0
- joint RJFT: limit lower=-3.1416 upper=3.1416 effort=1000 velocity=0.1 -> lower=-6.2832 upper=6.2832 effort=1000 velocity=0.1

Commit message: It seems that the dart kinematics work for correction/estimation
Former-commit-id: 0ac9c1a065979745292bd43c47b20a9db310aeff

File: compliance/scenes/KrangBlocks.urdf (robot description, URDF)
Before this commit: robot Krang, 23 links, 22 joints
Joints:
- joint LJFT: axis 0 1 0 -> 0 0 -1
- joint RJFT: axis 0 1 0 -> 0 0 -1
