Commit message: Trying to figure out whether dart computes com correctly
Former-commit-id: 834dcf3a76a6674356c3c7597280ba007cd851a2

File: common/scenes/testObject.urdf (robot description, URDF)
Before this commit: robot cylinder, 1 links, 0 joints
Links:
- link base_link: mass None -> 4.66; geometry collision box size=0.08 0.112 0.2025; visual box size=0.08 0.112 0.2025

Commit message: Got the com computation and visualization
Former-commit-id: 4b27f245f9005013ac3c44907191b63aa19e171d

File: common/scenes/testObject.urdf (robot description, URDF)
Before this commit: robot cylinder, 1 links, 0 joints
Links:
- removed link base_link
- added link Base, mass 1086.5; visual mesh filename=Spine/Tube.dae
