Commit message: Updated the urdf files to have the schunk grippers aligned with the bracket at degree 0
Former-commit-id: e0db7a47f924b0be5637b70fe2de2c409b86866b

File: common/scenes/Krang.urdf (robot description, URDF)
Before this commit: robot Krang, 23 links, 22 joints
Joints:
- joint LJFT: axis 0 1 0 -> 0 0 -1
- joint LMotorPlate1: origin xyz=0.02043 -0.04010 0.127 rpy=3.1416 0 2.04 -> xyz=-0.045 0.0 0.127 rpy=3.1416 0 0
- joint LMotorPlate2: origin xyz=-0.02043 0.04010 0.127 rpy=3.1416 0 -1.10 -> xyz=0.045 0.000 0.127 rpy=3.1416 0 3.1416
- joint RJFT: axis 0 1 0 -> 0 0 -1
- joint RMotorPlate1: origin xyz=0.02043 -0.04010 0.127 rpy=3.1416 0 2.04 -> xyz=-0.045 0.0 0.127 rpy=3.1416 0 0
- joint RMotorPlate2: origin xyz=-0.02043 0.04010 0.127 rpy=3.1416 0 -1.10 -> xyz=0.045 0.000 0.127 rpy=3.1416 0 3.1416

File: common/scenes/KrangBlocks.urdf (robot description, URDF)
Before this commit: robot Krang, 23 links, 22 joints
Joints:
- joint LMotorPlate1: origin xyz=0.02043 -0.04010 0.127 rpy=3.1416 0 2.04 -> xyz=-0.045 0.0 0.127 rpy=3.1416 0 0.0
- joint LMotorPlate2: origin xyz=-0.02043 0.04010 0.127 rpy=3.1416 0 -1.10 -> xyz=0.045 0.000 0.127 rpy=3.1416 0 3.1416
- joint RMotorPlate1: origin xyz=-0.02043 0.04010 0.127 rpy=3.1416 0 -1.10 -> xyz=-0.045 0.0 0.127 rpy=3.1416 0 0
- joint RMotorPlate2: origin xyz=0.050 0.1 0.0 rpy=1.57 3.1416 0 -> xyz=0.045 0.000 0.127 rpy=3.1416 0 3.1416

Commit message: 'Removed' the torso module from the model - if you want to put it back, uncomment the line in JTorso joint
Former-commit-id: 43a697acc67f8f79bad3b86ab8783c5d97939057

File: common/scenes/Krang.urdf (robot description, URDF)
Before this commit: robot Krang, 23 links, 22 joints
Joints:
- joint JTorso: origin xyz=-0.0285 0.584 0.1088 rpy=0 3.1416 0 -> xyz=-0.0285 0.443 0.1088 rpy=0 3.1416 0

File: common/scenes/KrangBlocks.urdf (robot description, URDF)
Before this commit: robot Krang, 23 links, 22 joints
Joints:
- joint JTorso: origin xyz=-0.0285 0.584 0.1088 rpy=0 3.1416 0 -> xyz=-0.0285 0.443 0.1088 rpy=0 3.1416 0

Commit message: Added an explanation to 01-dart and made the gripper plates fixed as opposed to prismatic in krang.urdf
Former-commit-id: 67945d1e35105c0748a94cbbe7256cc47278af74

File: common/scenes/Krang.urdf (robot description, URDF)
Before this commit: robot Krang, 23 links, 22 joints
Joints:
- joint LMotorPlate1: type prismatic -> fixed
- joint LMotorPlate2: type prismatic -> fixed

Commit message: Finished the com and mass details in Krang.urdf - need to put it in KrangBlocks and test on real robot
Former-commit-id: 86288aadcf29ef9c2a129bb0d89852c96bd0be9d

File: common/scenes/Krang.urdf (robot description, URDF)
Before this commit: robot Krang, 23 links, 22 joints
Links:
- link Base: mass 86.5 -> 81.856
- link Bracket: mass 3.11 -> 9.81
- link L1: mass 3.28 -> 3.836
- link L2: mass 3.76 -> 2.385
- link L3: mass 2.435 -> 2.306
- link L4: mass 2.356 -> 1.477
- link L5: mass 1.517 -> 1.369
- link L6: mass 1.428 -> 1.47
- link R1: mass 3.28 -> 3.836
- link R2: mass 3.76 -> 2.385
- link R3: mass 2.435 -> 2.306
- link R4: mass 2.356 -> 1.477
- link R5: mass 1.517 -> 1.369
- link R6: mass 1.428 -> 1.47
- link Spine: mass 6.547 -> 7.022
- link lGripper: mass 1.206 -> 2.3
- link rGripper: mass 1.206 -> 2.3

Commit message: Made changes to the Krang.urdf to separate the Kinect from the bracket
Former-commit-id: 81b32ac25c5a1ef4755d2d9361f1ecd52d1005d1

File: common/scenes/Krang.urdf (robot description, URDF)
Before this commit: robot Krang, 23 links, 22 joints
Links:
- added link Kinect, mass 0.705; collision box size=0.28 0.07 0.063; visual mesh filename=Kinect/Kinect.dae
- link Bracket: mass 9.81 -> 10.17; geometry collision box size=0.2815 0.23 0.22611; visual mesh filename=bracket.dae
Joints:
- added joint JKinect: type revolute, parent Bracket, child Kinect, origin xyz=-0.001 0.1805 -0.1120 rpy=3.1416 0 0, axis 1 0 0, limit lower=-3.1416 upper=3.1416 effort=1000 velocity=0.1

File: common/scenes/testObject.urdf (robot description, URDF)
Before this commit: robot cylinder, 1 links, 0 joints
Links:
- removed link Base
- added link Bracket, mass 9.81; collision box size=0.2815 0.23 0.22611; visual mesh filename=bracket.dae
- added link Kinect, mass 1086.5; collision box size=0.28 0.07 0.063; visual mesh filename=Kinect/Kinect.dae
Joints:
- added joint Joint: type revolute, parent Bracket, child Kinect, origin xyz=-0.001 0.1805 -0.1120 rpy=3.1416 0 0, axis 1 0 0, limit lower=-3.1416 upper=3.1416 effort=1000 velocity=0.1

Commit message: Changed the asserts in com grip visualization to while loops because we lose frames sometimes, added the torso in Krang.urdf (needs mass update), deleted krangblocks because no masses - needs to be redone
Former-commit-id: 3963d7a611afd6aedf39bce7aebd1eaffd5dcce1

File: common/scenes/Krang.urdf (robot description, URDF)
Before this commit: robot Krang, 24 links, 23 joints
Joints:
- joint JTorso: origin xyz=-0.0285 0.443 0.1088 rpy=0 3.1416 0 -> xyz=-0.0285 0.584 0.1088 rpy=0 3.1416 0

Commit message: Add the torso module to the mass model in the urdf file
Former-commit-id: 1664b45407b2c948979463878b65138ada25b854

File: common/scenes/Krang.urdf (robot description, URDF)
Before this commit: robot Krang, 24 links, 23 joints
Links:
- link Spine: mass 7.022 -> 10.302

Commit message: krang.urdf: relax the soft limits on the rotational joints in the arms
Former-commit-id: d64bf7f9d9ab3dc5dabc0e337d772ef564f89b45

File: common/scenes/Krang.urdf (robot description, URDF)
Before this commit: robot Krang, 24 links, 23 joints
Joints:
- joint LJ3: limit lower=-3.1416 upper=3.1416 effort=1000 velocity=0.1 -> lower=-4.7124 upper=4.7124 effort=1000 velocity=0.1
- joint LJ5: limit lower=-3.1416 upper=3.1416 effort=1000 velocity=0.1 -> lower=-4.7124 upper=4.7124 effort=1000 velocity=0.1; origin xyz=0 -0.2765 0 rpy=3.1416 3.1416 0 -> xyz=0 -0.2765 0 rpy=4.7124 4.7124 0
- joint LJ6: origin xyz=0 0 0 rpy=3.1416 3.1416 0 -> xyz=0 0 0 rpy=4.7124 4.7124 0
- joint LJFT: limit lower=-3.1416 upper=3.1416 effort=1000 velocity=0.1 -> lower=-4.7124 upper=4.7124 effort=1000 velocity=0.1; origin xyz=0 -0.200 0 rpy=1.5708 3.1416 0 -> xyz=0 -0.200 0 rpy=1.5708 4.7124 0
- joint RJ1: limit lower=-3.1416 upper=3.1416 effort=1000 velocity=0.1 -> lower=-4.7124 upper=4.7124 effort=1000 velocity=0.1
- joint RJ3: limit lower=-3.1416 upper=3.1416 effort=1000 velocity=0.1 -> lower=-4.7124 upper=4.7124 effort=1000 velocity=0.1; origin xyz=0 -0.328 0 rpy=-3.1416 -3.1416 0 -> xyz=0 -0.328 0 rpy=-4.7124 -4.7124 0
- joint RJ4: origin xyz=0 0 0 rpy=3.1416 3.1416 0 -> xyz=0 0 0 rpy=4.7124 4.7124 0
- joint RJ5: limit lower=-3.1416 upper=3.1416 effort=1000 velocity=0.1 -> lower=-4.7124 upper=4.7124 effort=1000 velocity=0.1; origin xyz=0 -0.2765 0 rpy=3.1416 3.1416 0 -> xyz=0 -0.2765 0 rpy=4.7124 4.7124 0
- joint RJ6: origin xyz=0 0 0 rpy=3.1416 3.1416 0 -> xyz=0 0 0 rpy=4.7124 4.7124 0
- joint RJFT: limit lower=-3.1416 upper=3.1416 effort=1000 velocity=0.1 -> lower=-4.7124 upper=4.7124 effort=1000 velocity=0.1; origin xyz=0 -0.200 0 rpy=1.5708 3.1416 0 -> xyz=0 -0.200 0 rpy=1.5708 4.7124 0
