Commit message: KrangBlocks.urdf contains the new data. Still to be tested
Former-commit-id: 9b08cceda0146a8d5df6d428ceca3cab4fcec5e9

File: common/scenes/KrangBlocksOld.urdf (robot description, URDF)
Before this commit: robot Krang, 24 links, 23 joints
Links:
- link Bracket: mass 6.533 -> 10.17
- link L1: mass 3.952 -> 3.836
- link L2: mass 3.925 -> 2.385
- link L3: mass 2.373 -> 2.306
- link L4: mass 2.373 -> 1.477
- link L5: mass 1.41334 -> 1.369
- link L6: mass 2.64634 -> 1.47
- link R1: mass 3.952 -> 3.836
- link R2: mass 3.925 -> 2.385
- link R3: mass 2.373 -> 2.306
- link R4: mass 2.373 -> 1.477
- link R5: mass 1.41334 -> 1.369
- link R6: mass 2.64634 -> 1.47
