Commit message: Added an infinitesmall mass to the plates so that the dart parser does not automatically add 0.1 kgs
Former-commit-id: 8e21cf65c9eb2e76a03f66b45088d16f8a84b6c5

File: common/scenes/KrangBlocks.urdf (robot description, URDF)
Before this commit: robot Krang, 24 links, 23 joints
Links:
- link lgPlate1: mass None -> 0.0001
- link lgPlate2: mass None -> 0.0001
- link rgPlate1: mass None -> 0.0001
- link rgPlate2: mass None -> 0.0001

Commit message: A few changes to the KrangBlkocks.urdf
Former-commit-id: 2d0ce294a6ac7d2d2a7b1885c17ad93dc64dd13c

File: common/scenes/KrangBlocks.urdf (robot description, URDF)
Before this commit: robot Krang, 24 links, 23 joints
Links:
- link Base: mass 81.856 -> 75.767
- link Spine: mass 10.302 -> 14.006; geometry collision box size=0.2340 0.59430 0.24097
